Commit message: Fix kitchen

File: mujoco_world/model/iai_kitchen_python.urdf (robot description, URDF)
Before this commit: robot iai_kitchen, 136 links, 135 joints
Links:
- link dining_area_jokkmokk_table_main: geometry collision mesh filename=package://iai_kitchen/meshes/jokkmokk/JokkmokkTable.obj; visual mesh filename=package://iai_kitchen/meshes/jokkmokk/JokkmokkTable.dae
