Commit message: Update iai_apartment

File: mujoco_world/model/iai_apartment/iai_apartment/meshes/apartment_unreal.urdf (robot description, URDF)
Before this commit: robot apartment, 120 links, 119 joints
Links:
- link armchair: geometry collision mesh filename=armchair.stl; visual mesh filename=package://iai_apartment/meshes/visual/armchair.dae
- link sofa: geometry collision mesh filename=sofa.stl; visual mesh filename=package://iai_apartment/meshes/visual/sofa.dae
Joints:
- joint armchair_joint: origin xyz=7.9688 -0.3791 0.0 rpy=0 0 1.9199 -> xyz=7.9688 -0.3791 0.3559428 rpy=0 0 1.9199
- joint bedside_table_joint: origin xyz=7.2110 0.1296 0.0 rpy=0 0 0 -> xyz=7.2110 0.1296 0.22990467 rpy=0 0 0
- joint cabinet2_door_handle_joint: origin xyz=0.25886013 -0.00184994 -0.05118866 rpy=0.0 0.0 1.5707963267948966 -> xyz=0.25886013 -0.00184994 -0.10518866 rpy=0.0 0.0 1.5707963267948966
- joint fridge_door1_handle_joint: origin xyz=0.46534321 -0.00799103 -0.4736869 rpy=0.0 0.0 1.5707963267948966 -> xyz=0.46534321 -0.00799103 -0.3616 rpy=0.0 0.0 1.5707963267948966
- joint fridge_door2_handle_joint: origin xyz=0.46538265 0.00804657 0.28486839 rpy=0.0 0.0 1.5707963267948966 -> xyz=0.46538265 0.00804657 0.31786839 rpy=0.0 0.0 1.5707963267948966
- joint kitchen2_root_joint: origin xyz=0.0 0.0 0.0 -> xyz=0.1 0.0 0.0
- joint sofa_joint: origin xyz=8.1986 2.4096 0.0 rpy=0 0 0 -> xyz=8.1986 2.4096 0.35732983 rpy=0 0 0
