Commit message: Add left window

File: mujoco_world/model/iai_apartment/iai_apartment_with_window4/meshes/apartment_unreal_with_window4.urdf (robot description, URDF)
Before this commit: robot apartment, 123 links, 122 joints
Links:
- added link window4_right; collision box size=0.843426 0.02 2.05976; visual mesh filename=package://iai_apartment/meshes/unreal/SM_Window_Right.dae
- added link window4_right_handle; collision cylinder length=0.052952 radius=0.008; collision cylinder length=0.075236 radius=0.008
Joints:
- added joint window4_right_handle_joint: type revolute, parent window4_right, child window4_right_handle, origin xyz=-0.823253 -0.026228 0.0, axis 0 -1 0, limit lower=0.0 upper=3.141592653589793 effort=1000.0 velocity=3.141592653589793
- added joint window4_right_joint: type revolute, parent window4_frame, child window4_right, origin xyz=0.924416 -0.00162 -0.42549, axis 0 0 1, limit lower=0.0 upper=1.5708 effort=1000.0 velocity=1.5708
- joint window4_left_handle_joint: origin xyz=-0.823253 -0.026228 0.0 -> xyz=0.823253 -0.026228 0.0
- joint window4_left_joint: axis 0 0 1 -> 0 0 -1; origin xyz=0.924416 -0.00162 -0.42549 -> xyz=-0.9369 0.00162 -0.42549

Commit message: Fix window meshes

File: mujoco_world/model/iai_apartment/iai_apartment_with_window4/meshes/apartment_unreal_with_window4.urdf (robot description, URDF)
Before this commit: robot apartment, 125 links, 124 joints
Links:
- link window4_left: geometry collision box size=0.86406 0.02 2.0631; visual mesh filename=package://iai_apartment/meshes/unreal/SM_Window_Left.dae
- link window4_right: geometry collision box size=0.843426 0.02 2.0631; visual mesh filename=package://iai_apartment/meshes/unreal/SM_Window_Right.dae
Joints:
- joint window4_left_handle_joint: origin xyz=0.823253 -0.026228 0.0 -> xyz=0.834107 -0.019236 0.0
- joint window4_left_joint: origin xyz=-0.9369 0.00162 -0.42549 -> xyz=-0.929112 0.00162 -0.425471
- joint window4_right_handle_joint: origin xyz=-0.823253 -0.026228 0.0 -> xyz=-0.815383 -0.019236 0.0
- joint window4_right_joint: origin xyz=0.924416 -0.00162 -0.42549 -> xyz=0.916552 0 -0.425471
