Commit message: Update box

File: mujoco_world/model/box/urdf/box.urdf (robot description, URDF)
Before this commit: robot box, 3 links, 2 joints
Links:
- removed link box_top_layer_bottom
- removed link box_top_layer_top
- added link box_flap_side_1; collision mesh filename=package://mujoco_world/model/box/urdf/meshes/BoxFlapSide1.s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; visual mesh filename=package://mujoco_world/model/box/urdf/meshes/BoxFlapSide1.d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
- added link box_flap_side_2; collision mesh filename=package://mujoco_world/model/box/urdf/meshes/BoxFlapSide2.s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; visual mesh filename=package://mujoco_world/model/box/urdf/meshes/BoxFlapSide2.d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
Joints:
- removed joint box_top_layer_bottom_joint
- removed joint box_top_layer_top_joint
- added joint box_flap_side_1_joint: type continuous, parent box_body, child box_flap_side_1, origin xyz=-0.17 0 0.168 rpy=0 0 0, axis 0 -1 0
- added joint box_flap_side_2_joint: type continuous, parent box_body, child box_flap_side_2, origin xyz=0.17 0 0.166 rpy=0 0 0, axis 0 1 0
